Commit message: fix code

File: realsense-ros/realsense2_description/urdf/_d435.urdf.xacro (robot description, xacro)
@@ -66,5 +66,5 @@
           <origin xyz="${d435_zero_depth_to_glass + d435_glass_to_front} ${-d435_cam_depth_py} 0" rpy="${M_PI/2} 0 ${M_PI/2}"/>
           <geometry>
-            <mesh filename="file:///home/jy/colcon_ws/src/realsense-ros/realsense2_description/meshes/d435.dae" scale="1 1 1"/>
+            <mesh filename="package://realsense2_description/meshes/d435.dae" scale="1 1 1"/>
           </geometry>
         </xacro:if>
